File: MXM.kicad_sch (KiCad schematic)
At the start: 9 parts

Commit message: update readme.md
Other:
- company: (none) -> mothenjoyer69
- title: (none) -> ThunderMXM
- moved on the sheet: C17, C18, C19, C20, C21, C22, C23, C6, MXM1
