File: m2-tb3.kicad_sch (KiCad schematic)
At the start: 10 parts, among them J7 M.2_1_USB, J8 M.2_2_PCIE

Commit message: update readme.md
Other:
- note added: "M.2-A (USB)"
- note added: "M.2-B (PCIe)"
- note added: "Power caps"
- company: (none) -> mothenjoyer69
- title: (none) -> ThunderMXM
- moved on the sheet: C1, C2, C3, C4, C5, J7, J8, R1, R2, R3
