File: tb3-mxm.kicad_sch (KiCad schematic)
At the start: 5 parts

Commit message: update readme.md
Other:
- note added: "ThunderMXM"
- note added: "To-do: - Finish schematics!!! - Finalize layout - Route it all - Stop being lazy and just route it all"
- company: (none) -> mothenjoyer69
- title: (none) -> ThunderMXM
- moved on the sheet: H1, H2, H3, H4, H5
